File: apu_mega_shield.brd (EAGLE design)
At the start: 105.4 x 53.6 mm, 36 parts, among them IC1 74HCT573D, IC2 4050D, IC3 DS1307, Q1 32.768, U1 IS62C1024AL-35QLI, X1 MICROSD

Commit message: Micro SD card detect pullup resistor added.
Parts:
- C1, C2, C7: device resistor:C0603 -> rcl:C0805
- RN1: device resistor-net:RN-9 -> resistor-net:RN-10
Connections:
- net CD: now also RN1.10
Routing:
- net GND: track 264.2 -> 180.9 mm
- net VCC: track 252.5 -> 205.8 mm, vias 0 -> 1
- net RST: track 163.1 -> 126.6 mm, vias 0 -> 3
- net D0: track 81.6 -> 114.8 mm
- net CD: track 30.5 -> 56.9 mm
- net D3: track 94.2 -> 76.8 mm
- net !RD: track 104.9 -> 88.3 mm, vias 2 -> 3
- net LEFT: track 65.1 -> 80.6 mm
- net DOWN: track 64.5 -> 53.1 mm, vias 0 -> 1
- net D6: track 79.8 -> 69.1 mm, vias 0 -> 1
- net D1: track 88.5 -> 80.5 mm, vias 0 -> 1
- net A10: track 133.9 -> 126.3 mm, vias 0 -> 1
- net A11: track 89.9 -> 82.8 mm, vias 0 -> 2
- net D7: track 77.8 -> 71.1 mm, vias 0 -> 1
- net A16: track 15.4 -> 9.70 mm
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