File: PCB/apu_pcb.brd (EAGLE design)
At the start: 72.4 x 62.2 mm, 34 parts, among them IC1 S-SMP, IC2 S-DSP, IC3 5x832 SRAM, IC4 5x832 SRAM, IC5 DAC, IC6 LM2904

Commit message: Improvements on the pc application
Routing:
- net LRCK: track 65.8 -> 63.7 mm
- net SO: track 64.0 -> 62.0 mm
- net BCK: track 50.9 -> 52.4 mm
- net !RESET: track 39.6 -> 38.7 mm
- net VCC: track 215.6 -> 216.2 mm
- net GND: vias 57 -> 61
