File: PCB/apu_mega_shield.sch (EAGLE design)
At the start: 39 parts, among them IC1 74AHC573, IC2 4050D, IC3 DS1307, IC4 LP298XS, Q1 32.768, U1 IS62C1024AL, X1 MICROSDMOLEX

Commit message: All parts that are not buttons or connectors replaced with SMT equivalents. :)
Parts:
- removed RN1: 10K, resistor-net:RN09
- added R10, R11, R12, R13, R14, R15, R2, R3, R7: 10K, resistor:R-US_R0805
- BAT: device adafruit:CR1220THM -> adafruit:CR1220SMT
- C3, C4, C5, C6: device rcl-ez:C-US025-025X050 -> resistor:C-EUC0805
- IC3: device adafruit:DS1307 -> adafruit:DS1307SMT
- Q1: device crystal:CRYTALTC38H -> crystal:CRYTALSMD
- R1, R8, R9: device adafruit:R-US_0207/10 -> resistor:R-US_R0805
- R4, R5: device rcl:R-US_0207/10 -> resistor:R-US_R0805
Connections:
- removed net N$12: IC2B.O, X1.DATA_IN
- removed net N$39: BAT.+1, IC3.VBAT
- removed net N$5: ACT.A, IC2D.O
- removed net N$6: IC2A.O, X1.SCLK
- removed net N$7: IC2C.O, R6.1, X1.CS
- new net BUF_CLK: IC2D.O, X1.SCLK
- new net BUF_CS: IC2F.O, R6.1, X1.CS
- new net BUF_DI: IC2E.O, X1.DATA_IN
- new net BUF_LED: ACT.A, IC2A.O
- new net N$15: BAT.+, IC3.VBAT
- net !RD: now also R14.2; no longer RN1.4
- net !WR: now also R15.2; no longer RN1.3
- net CD: now also R3.2; no longer RN1.10
- net CS: now also IC2F.I; no longer IC2C.I
- net DI: now also IC2E.I; no longer IC2B.I
- net DOWN: now also R11.2; no longer RN1.7
- net GND: now also IC2B.I, IC2C.I; no longer IC2E.I, IC2F.I
- net LEFT: now also R13.2; no longer RN1.5
- net RIGHT: now also R10.2; no longer RN1.8
- net RST: now also R2.2; no longer RN1.2
- net SELECT: now also R7.2; no longer RN1.9
- net UP: now also R12.2; no longer RN1.6
- net VCC: now also R10.1, R11.1, R12.1, R13.1, R14.1, R15.1, R2.1, R3.1, R7.1; no longer RN1.1
Other:
- moved on the sheet: APU, DOWN, IC2A, IC2B, IC2C, IC2D, IC2E, IC2F, LEFT, RIGHT, SELECT, UP

Commit message: R1 removed from PCB. It was supposed to be the current limiting resistor for the LCD backlight, however, the LCD module in use already has a current limiting resistor mounted right on that module.
Parts:
- removed R1: 220, resistor:R-US_R0805
Connections:
- net N$14: now also U$6.46; no longer R1.2
- net VCC: no longer R1.1
Changed lines of the file:
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@@
 <part name="SUPPLY2" library="supply2" deviceset="GND" device=""/>
 <part name="X1" library="adafruit" deviceset="MICROSD" device="MOLEX"/>
-<part name="R1" library="resistor" deviceset="R-US_" device="R0805" value="220"/>
 <part name="R2" library="resistor" deviceset="R-US_" device="R0805" value="10K"/>
 <part name="R3" library="resistor" deviceset="R-US_" device="R0805" value="10K"/>
@@
 <instance part="SUPPLY2" gate="GND" x="383.54" y="-15.24"/>
 <instance part="X1" gate="G$1" x="353.06" y="15.24"/>
-<instance part="R1" gate="G$1" x="233.68" y="121.92" rot="R270"/>
 <instance part="R2" gate="G$1" x="142.24" y="10.16" rot="R270"/>
 <instance part="R3" gate="G$1" x="182.88" y="10.16" rot="R270"/>
@@
 <wire x1="243.84" y1="114.3" x2="243.84" y2="116.84" width="0.1524" layer="91"/>
 <label x="256.54" y="134.62" size="1.778" layer="95"/>
-<pinref part="R1" gate="G$1" pin="1"/>
-<wire x1="233.68" y1="127" x2="243.84" y2="127" width="0.1524" layer="91"/>
-<junction x="243.84" y="127"/>
 </segment>
 <segment>
@@
 <segment>
 <pinref part="JP1" gate="A" pin="15"/>
-<pinref part="R1" gate="G$1" pin="2"/>
 <wire x1="233.68" y1="111.76" x2="233.68" y2="116.84" width="0.1524" layer="91"/>
-</segment>
-</net>
+<wire x1="233.68" y1="116.84" x2="251.46" y2="116.84" width="0.1524" layer="91"/>
+<wire x1="251.46" y1="116.84" x2="251.46" y2="101.6" width="0.1524" layer="91"/>
+<pinref part="U$6" gate="G$1" pin="46"/>
+<wire x1="251.46" y1="101.6" x2="259.08" y2="101.6" width="0.1524" layer="91"/>
+</segment>
+</net>

Commit message: Final revisions to the PCB design, hopefully. :)
Parts:
- added C9: 100nF, apu_pcb:C0805
- C1, C2, C7: device rcl:C-EUC0805 -> apu_pcb:C0805
- C3, C4, C5, C6: device resistor:C-EUC0805 -> apu_pcb:C0805
- R10, R11, R12, R13, R14, R15, R2, R3, R4, R5, R7, R8, R9: device resistor:R-US_R0805 -> adafruit:R-US_R0805
Connections:
- net A11: now also U1.A14; no longer U1.A16
- net A13: now also U1.A12; no longer U1.A14
- net A17: now also U1.A16; no longer U1.A12
- net GND: now also C9.1
- net VCC: now also C9.2
Other:
- moved on the sheet: C1, C2, C3, C4, C5, C6, C7
